File: hardware/Bald Probe Test Fixture rev1.kicad_sch (KiCad schematic)
At the start: 0 parts

Commit message: schematic and pcb. need to setup board rules
Parts:
- added J1: SMA_IN, Connector_Coaxial:SMA_Molex_73251-1153_EdgeMount_Horizontal, symbol Connector:Conn_Coaxial
- added J2: SMA_OUT, Connector_Coaxial:SMA_Molex_73251-1153_EdgeMount_Horizontal, symbol Connector:Conn_Coaxial
Connections:
- new net GND: J1.2 (Ext), J2.2 (Ext)
- new net thru_trace: J1.1 (In), J2.1 (In)

Commit message: rev1 ready for fab
Other:
- note added: "Using Molex 73251-1153. Footprint is close to existing stock but not exact."
- title: Bald Probe Test Fixtures -> Bald Probe Test Fixture (SMA)
Changed lines of the file:
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@@
 	(paper "A4")
 	(title_block
-		(title "Bald Probe Test Fixtures")
+		(title "Bald Probe Test Fixture (SMA)")
+		(date "2024-07-05")
 		(rev "1")
 		(company "@baldengineer")
@@
 		)
 	)
+	(text "Using Molex 73251-1153. \nFootprint is close to existing stock but not exact."
+		(exclude_from_sim no)
+		(at 119.38 83.82 0)
+		(effects
+			(font
+				(size 1.27 1.27)
+			)
+		)
+	)
